File: motorboard.brd (EAGLE design)
At the start: 69.5 x 24.5 mm, 21 parts, among them U1 STM32F302_303C2

Commit message: fixed capacitors values
Parts:
- C4: value 4.7uF -> 10uF
- C5: value 10uF -> 100nF
Changed lines of the file:
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@@
 <attribute name="NAME" x="34.93" y="20.93" size="1.27" layer="26" rot="MR180"/>
 </element>
-<element name="C4" library="resistor" package="C0805" value="4.7uF" x="25.7" y="11.2" smashed="yes" rot="R90">
+<element name="C4" library="resistor" package="C0805" value="10uF" x="25.7" y="11.2" smashed="yes" rot="R90">
 <attribute name="NAME" x="26.77" y="8.93" size="1.27" layer="25" rot="R180"/>
 </element>
-<element name="C5" library="resistor" package="C0805" value="10uF" x="31" y="19.2" smashed="yes" rot="MR180">
+<element name="C5" library="resistor" package="C0805" value="100nF" x="31" y="19.2" smashed="yes" rot="MR180">
 <attribute name="NAME" x="26.73" y="19.73" size="1.27" layer="26" rot="MR180"/>
 </element>
